File: ac-dc-converter/ac-dc-converter.kicad_pcb (KiCad board)
At the start: 2 copper layers, 100 x 50 mm, 23 parts, among them J1 726386-2, J2 726386-2, J3 726386-2, J4 726386-2, J5 726386-2, J7 SPM1502SJ, J8 726386-2

Commit message: .
Connections:
- C1 pad 1: ACH -> ACL
- C1 pad 2: ACL -> ACN
- FL1 pad 1: ACH -> ACL
- FL1 pad 3: ACL -> ACN
- J3 pad 1: ACH -> ACL
- J3 pad 2: ACH -> ACL
- J4 pad 1: ACL -> ACN
- J4 pad 2: ACL -> ACN
- RV2 pad 1: ACH -> ACL
- RV2 pad 2: ACL -> ACN
Routing:
- net ACH: track 79.7 -> 0.00 mm
- net ACN: track 0.00 -> 55.6 mm
- net ACL: track 55.6 -> 79.7 mm
Other:
- board text added: "L"
- board text added: "N"
Changed lines of the file:
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@@
 	(net 0 "")
 	(net 1 "GND")
-	(net 2 "ACH")
+	(net 2 "ACN")
 	(net 3 "+15V")
 	(net 4 "+170V")
@@
 			(layers "*.Cu" "*.Mask")
 			(remove_unused_layers no)
-			(net 2 "ACH")
+			(net 13 "ACL")
 			(pinfunction "1")
 			(pintype "passive")
@@
 			(layers "*.Cu" "*.Mask")
 			(remove_unused_layers no)
-			(net 13 "ACL")
+			(net 2 "ACN")
 			(pinfunction "3")
 			(pintype "passive")
@@
 			(layers "*.Cu" "*.Mask")
 			(remove_unused_layers no)
-			(net 2 "ACH")
+			(net 13 "ACL")
 			(pintype "passive")
 		)
@@
 			(layers "*.Cu" "*.Mask")
 			(remove_unused_layers no)
-			(net 13 "ACL")
+			(net 2 "ACN")
 			(pintype "passive")
 		)
@@
 			(layers "*.Cu" "*.Mask")
 			(remove_unused_layers no)
-			(net 13 "ACL")
+			(net 2 "ACN")
 			(pinfunction "1")
 			(pintype "unspecified")
@@
 			(layers "*.Cu" "*.Mask")
 			(remove_unused_layers no)
-			(net 13 "ACL")
+			(net 2 "ACN")
 			(pinfunction "2")
 			(pintype "unspecified")
@@
 			(layers "*.Cu" "*.Mask")
 			(remove_unused_layers no)
-			(net 2 "ACH")
+			(net 13 "ACL")
 			(pinfunction "1")
 			(pintype "unspecified")
@@
 			(layers "*.Cu" "*.Mask")
 			(remove_unused_layers no)
-			(net 2 "ACH")
+			(net 13 "ACL")
 			(pinfunction "2")
 			(pintype "unspecified")
@@
 			(layers "*.Cu" "*.Mask")
 			(remove_unused_layers no)
-			(net 2 "ACH")
+			(net 13 "ACL")
 			(pintype "passive")
 		)
@@
 			(layers "*.Cu" "*.Mask")
 			(remove_unused_layers no)
-			(net 13 "ACL")
+			(net 2 "ACN")
 			(pintype "passive")
 		)
@@
 		)
 	)
+	(gr_text "N"
+		(at 32.05 55.55 0)
+		(layer "F.SilkS")
+		(effects
+			(font
+				(size 2 2)
+				(thickness 0.5)
+				(bold yes)
+			)
+			(justify left bottom)
+		)
+	)
+	(gr_text "L"
+		(at 32.37 67.74 0)
+		(layer "F.SilkS")
+		(effects
+			(font
+				(size 2 2)
+				(thickness 0.5)
+				(bold yes)
+			)
+			(justify left bottom)
+		)
+	)
 	(gr_text "+170V"
 		(at 116.880001 83.867834 90)
@@
 	)
 	(segment
-		(start 54.92 36.96)
-		(end 58.96 41)
-		(width 2)
-		(layer "B.Cu")
-		(net 2)
-	)
-	(segment
-		(start 42.98 49.97)
-		(end 46.91 46.04)
-		(width 2)
-		(layer "B.Cu")
-		(net 2)
-	)
-	(segment
-		(start 50.31 74.14105)
-		(end 47.36105 77.09)
+		(start 50.31 59.91)
+		(end 55.01 64.61)
 		(width 2)
 		(layer "B.Cu")
@@
 	)
 	(segment
-		(start 50.31 66.64)
-		(end 50.31 74.14105)
+		(start 55.01 67.86)
+		(end 62.34705 75.19705)
 		(width 2)
 		(layer "B.Cu")
@@
 	)
 	(segment
-		(start 37.12 66.64)
-		(end 50.31 66.64)
+		(start 50.26 59.86)
+		(end 50.26 59.31)
 		(width 2)
 		(layer "B.Cu")
@@
 	)
 	(segment
-		(start 35.65 66.64)
-		(end 33.04 64.03)
+		(start 52.055 61.655)
+		(end 50.26 59.86)
 		(width 2)
 		(layer "B.Cu")
@@
 	)
 	(segment
-		(start 46.91 39.25)
-		(end 49.2 36.96)
+		(start 51.955 61.655)
+		(end 52.055 61.655)
 		(width 2)
 		(layer "B.Cu")
@@
 	)
 	(segment
-		(start 33.04 64.03)
-		(end 33.04 52.34)
+		(start 36.94 54.36)
+		(end 44.66 54.36)
 		(width 2)
 		(layer "B.Cu")
@@
 	)
 	(segment
-		(start 33.04 52.34)
-		(end 35.41 49.97)
+		(start 55.01 64.61)
+		(end 55.01 67.86)
 		(width 2)
 		(layer "B.Cu")
@@
 	)
 	(segment
-		(start 37.12 66.64)
-		(end 35.65 66.64)
+		(start 62.34705 75.19705)
+		(end 62.34705 77.09)
 		(width 2)
 		(layer "B.Cu")
@@
 	)
 	(segment
-		(start 46.91 46.04)
-		(end 46.91 39.25)
+		(start 44.66 54.36)
+		(end 51.955 61.655)
 		(width 2)
 		(layer "B.Cu")
@@
 	)
 	(segment
-		(start 35.41 49.97)
-		(end 42.98 49.97)
+		(start 50.31 48.65)
+		(end 50.31 59.91)
 		(width 2)
 		(layer "B.Cu")
@@
 	)
 	(segment
-		(start 49.2 36.96)
-		(end 54.92 36.96)
+		(start 50.96 48)
+		(end 50.31 48.65)
 		(width 2)
 		(layer "B.Cu")
@@
 	)
 	(segment
-		(start 50.31 59.91)
-		(end 55.01 64.61)
+		(start 54.92 36.96)
+		(end 58.96 41)
 		(width 2)
 		(layer "B.Cu")
@@
 	)
 	(segment
-		(start 55.01 67.86)
-		(end 62.34705 75.19705)
+		(start 42.98 49.97)
+		(end 46.91 46.04)
 		(width 2)
 		(layer "B.Cu")
@@
 	)
 	(segment
-		(start 50.26 59.86)
-		(end 50.26 59.31)
+		(start 50.31 74.14105)
+		(end 47.36105 77.09)
 		(width 2)
 		(layer "B.Cu")
@@
 	)
 	(segment
-		(start 52.055 61.655)
-		(end 50.26 59.86)
+		(start 50.31 66.64)
+		(end 50.31 74.14105)
 		(width 2)
 		(layer "B.Cu")
@@
 	)
 	(segment
-		(start 51.955 61.655)
-		(end 52.055 61.655)
+		(start 37.12 66.64)
+		(end 50.31 66.64)
 		(width 2)
 		(layer "B.Cu")
@@
 	)
 	(segment
-		(start 36.94 54.36)
-		(end 44.66 54.36)
+		(start 35.65 66.64)
+		(end 33.04 64.03)
 		(width 2)
 		(layer "B.Cu")
@@
 	)
 	(segment
-		(start 55.01 64.61)
-		(end 55.01 67.86)
+		(start 46.91 39.25)
+		(end 49.2 36.96)
 		(width 2)
 		(layer "B.Cu")
@@
 	)
 	(segment
-		(start 62.34705 75.19705)
-		(end 62.34705 77.09)
+		(start 33.04 64.03)
+		(end 33.04 52.34)
 		(width 2)
 		(layer "B.Cu")
@@
 	)
 	(segment
-		(start 44.66 54.36)
-		(end 51.955 61.655)
+		(start 33.04 52.34)
+		(end 35.41 49.97)
 		(width 2)
 		(layer "B.Cu")
@@
 	)
 	(segment
-		(start 50.31 48.65)
-		(end 50.31 59.91)
+		(start 37.12 66.64)
+		(end 35.65 66.64)
 		(width 2)
 		(layer "B.Cu")
@@
 	)
 	(segment
-		(start 50.96 48)
-		(end 50.31 48.65)
+		(start 46.91 46.04)
+		(end 46.91 39.25)
+		(width 2)
+		(layer "B.Cu")
+		(net 13)
+	)
+	(segment
+		(start 35.41 49.97)
+		(end 42.98 49.97)
+		(width 2)
+		(layer "B.Cu")
+		(net 13)
+	)
+	(segment
+		(start 49.2 36.96)
+		(end 54.92 36.96)
 		(width 2)
 		(layer "B.Cu")
