File: ac-dc-converter/ac-dc-converter.kicad_sch (KiCad schematic)
At the start: 19 parts, among them J1 726386-2, J2 726386-2, J3 726386-2, J4 726386-2, J5 726386-2, J7 SPM1502SJ, J8 726386-2

Commit message: .
Connections:
- net ACH is gone; now on net ACL: C1.1, FL1.1, J3.1, J3.2, RV2.1
- net ACL: no longer C1.2, FL1.3, J4.1, J4.2, RV2.2
- new net ACN: C1.2, FL1.3, J4.1, J4.2, RV2.2
Changed lines of the file:
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@@
 			)
 		)
-		(property "Value" "ACL"
+		(property "Value" "ACN"
 			(at 85.09 93.9799 90)
 			(effects
@@
 			)
 		)
-		(property "Value" "ACH"
+		(property "Value" "ACL"
 			(at 85.09 82.5499 90)
 			(effects
@@
 			)
 		)
-		(property "Value" "ACL"
+		(property "Value" "ACN"
 			(at 35.56 48.2599 90)
 			(effects
@@
 			)
 		)
-		(property "Value" "ACH"
+		(property "Value" "ACL"
 			(at 35.56 30.4799 90)
 			(effects
